File: Project/EEEEagle/smallDevV1.sch (EAGLE design)
At the start: 25 parts, among them IC1 TLC272D

Commit message: commit yo
Parts:
- removed AUDIOJACK: (no value), myLibrary:M041.27MM
- removed R1: 1K, adafruit:R-US_M0805
- removed R7: 20K, adafruit:R-US_M0805
- removed SOS: (no value), SparkFun-Electromechanical:SWITCH-SPDT-SMD-A
- removed U$2: AUDIO-JACK3, SparkFun-Connectors:AUDIO-JACK3
- added JP1: Microphone, SparkFun-Connectors:M03LOCK
- added R11: 1K, adafruit:R-US_M0805
- added SOS_INDICATOR2: (no value), adafruit:LEDCHIP-LED0805
- added U$3: SWITCH_SPDT, myLibrary:SWITCH_SPDT
- 3.3V: device SparkFun-Boards:ARDUINO_PRO_MINI -> myLibrary:ARDUINO_PRO_MINI
- U$1: value (none) -> 10K
Connections:
- removed net BLEH: 3.3V.2
- removed net N$10: R1.1, SOS_INDICATOR1.A
- removed net N$11: 3.3V.13
- removed net N$12: 3.3V.12
- removed net N$2: AUDIOJACK.4, IC1B.-IN, R2.1
- removed net N$5: 3.3V.RX1
- removed net N$7: AUDIOJACK.2, R5.1, R6.2, R7.2
- removed net N$9: SOS.S, SOS_INDICATOR1.C
- new net LED: 3.3V.13, R11.1
- new net MICROPHONE: JP1.2, R5.1, R6.2
- new net N$1: R11.2, SOS_INDICATOR1.A, SOS_INDICATOR2.A
- new net SPEAKER_R: IC1B.-IN, JP1.1, R2.1
- net BUTTON: now also 3.3V.A7
- net GND: now also JP1.3, SOS_INDICATOR1.C, SOS_INDICATOR2.C, U$3.O; no longer AUDIOJACK.1, R7.1, SOS.O
- net SPEAKER: now also 3.3V.5; no longer 3.3V.A6
- net SWITCH: now also U$3.P; no longer SOS.P
- net VCC: no longer R1.2
Other:
- moved on the sheet: R5, SOS_INDICATOR1
